Commit message: Fix old name

File: cookobot_gazebo/robot_description/urdf/arm_hardware.xacro (robot description, xacro)
@@ -33,5 +33,5 @@
         <origin xyz="-0.028 -0.0493 0.014" rpy="0.0 0.0 -${M_PI/2}"/>
         <geometry>
-          <mesh filename="package://cookobot-arm/meshes/mount.stl" scale="${M_SCALE} ${M_SCALE} ${M_SCALE}"/>
+          <mesh filename="package://cookobot_gazebo/meshes/mount.stl" scale="${M_SCALE} ${M_SCALE} ${M_SCALE}"/>
         </geometry>
         <material name="${color}"/>
@@ -61,5 +61,5 @@
         <origin xyz=" 0 0 0 " rpy="0 0 0"/>
         <geometry>
-          <mesh filename="package://cookobot-arm/meshes/turtlebot_finger.stl" scale="${M_SCALE} ${M_SCALE} ${M_SCALE}"/>
+          <mesh filename="package://cookobot_gazebo/meshes/turtlebot_finger.stl" scale="${M_SCALE} ${M_SCALE} ${M_SCALE}"/>
         </geometry>
         <material name="${color}"/>
@@ -95,5 +95,5 @@
         <origin xyz=" 0 0 0 " rpy="0 0 0"/>
         <geometry>
-          <mesh filename="package://cookobot-arm/meshes/ax12_box.stl" scale="${M_SCALE} ${M_SCALE} ${M_SCALE}"/>
+          <mesh filename="package://cookobot_gazebo/meshes/ax12_box.stl" scale="${M_SCALE} ${M_SCALE} ${M_SCALE}"/>
         </geometry>
         <material name="Black"/>
@@ -123,5 +123,5 @@
         <origin xyz=" 0 0 0 " rpy="0 0 0"/>
         <geometry>
-          <mesh filename="package://cookobot-arm/meshes/F10.stl" scale="${M_SCALE} ${M_SCALE} ${M_SCALE}"/>
+          <mesh filename="package://cookobot_gazebo/meshes/F10.stl" scale="${M_SCALE} ${M_SCALE} ${M_SCALE}"/>
         </geometry>
         <material name="${color}"/>
@@ -151,5 +151,5 @@
         <origin xyz=" 0 0 0 " rpy="0 0 0"/>
         <geometry>
-          <mesh filename="package://cookobot-arm/meshes/F3.stl" scale="${M_SCALE} ${M_SCALE} ${M_SCALE}"/>
+          <mesh filename="package://cookobot_gazebo/meshes/F3.stl" scale="${M_SCALE} ${M_SCALE} ${M_SCALE}"/>
         </geometry>
         <material name="${color}"/>
@@ -182,5 +182,5 @@
         <origin xyz=" 0 0 0 " rpy="0 0 0"/>
         <geometry>
-          <mesh filename="package://cookobot-arm/meshes/F3.stl" scale="${M_SCALE} ${M_SCALE} ${M_SCALE}"/>
+          <mesh filename="package://cookobot_gazebo/meshes/F3.stl" scale="${M_SCALE} ${M_SCALE} ${M_SCALE}"/>
         </geometry>
         <material name="${color}"/>
@@ -213,5 +213,5 @@
         <origin xyz=" 0 0 0 " rpy="0 0 0"/>
         <geometry>
-          <mesh filename="package://cookobot-arm/meshes/F2.stl" scale="${M_SCALE} ${M_SCALE} ${M_SCALE}"/>
+          <mesh filename="package://cookobot_gazebo/meshes/F2.stl" scale="${M_SCALE} ${M_SCALE} ${M_SCALE}"/>
         </geometry>
         <material name="${color}"/>
@@ -244,5 +244,5 @@
         <origin xyz=" 0 0 0 " rpy="0 0 0"/>
         <geometry>
-          <mesh filename="package://cookobot-arm/meshes/F4.stl" scale="${M_SCALE} ${M_SCALE} ${M_SCALE}"/>
+          <mesh filename="package://cookobot_gazebo/meshes/F4.stl" scale="${M_SCALE} ${M_SCALE} ${M_SCALE}"/>
         </geometry>
         <material name="${color}"/>
@@ -272,5 +272,5 @@
         <origin xyz="0.016 0 -.015 " rpy="${M_PI} ${-M_PI/2} ${M_PI/2}"/>
         <geometry>
-          <mesh filename="package://cookobot-arm/meshes/pincher_finger_base.stl" scale=".01 .01 .01"/>
+          <mesh filename="package://cookobot_gazebo/meshes/pincher_finger_base.stl" scale=".01 .01 .01"/>
         </geometry>
         <material name="${color}"/>
@@ -295,5 +295,5 @@
         <xacro:insert_block name="origin"/>
         <geometry>
-          <mesh filename="package://cookobot-arm/meshes/pincher_finger.stl" scale=".01 .01 .01"/>
+          <mesh filename="package://cookobot_gazebo/meshes/pincher_finger.stl" scale=".01 .01 .01"/>
         </geometry>
         <material name="${color}"/>

File: cookobot_gazebo/robot_description/urdf/turtlebot3_burger_arm.urdf.xacro (robot description, xacro)
@@ -36,5 +36,5 @@
       <origin xyz="-0.032 0 0.0" rpy="0 0 0"/>
       <geometry>
-        <mesh filename="file://$(find cookobot-arm)/robot_description/urdf/meshes/bases/burger_base.stl" scale="0.001 0.001 0.001"/>
+        <mesh filename="file://$(find cookobot_gazebo)/robot_description/urdf/meshes/bases/burger_base.stl" scale="0.001 0.001 0.001"/>
       </geometry>
       <material name="light_black"/>
@@ -64,5 +64,5 @@
       <origin xyz="0 0 0" rpy="1.57 0 0"/>
       <geometry>
-        <mesh filename="file://$(find cookobot-arm)/robot_description/urdf/meshes/wheels/left_tire.stl" scale="0.001 0.001 0.001"/>
+        <mesh filename="file://$(find cookobot_gazebo)/robot_description/urdf/meshes/wheels/left_tire.stl" scale="0.001 0.001 0.001"/>
       </geometry>
       <material name="dark"/>
@@ -92,5 +92,5 @@
       <origin xyz="0 0 0" rpy="1.57 0 0"/>
       <geometry>
-        <mesh filename="file://$(find cookobot-arm)/robot_description/urdf/meshes/wheels/right_tire.stl" scale="0.001 0.001 0.001"/>
+        <mesh filename="file://$(find cookobot_gazebo)/robot_description/urdf/meshes/wheels/right_tire.stl" scale="0.001 0.001 0.001"/>
       </geometry>
       <material name="dark"/>
@@ -145,5 +145,5 @@
       <origin xyz="0 0 0.0" rpy="0 0 0"/>
       <geometry>
-        <mesh filename="file://$(find cookobot-arm)/robot_description/urdf/meshes/sensors/lds.stl" scale="0.001 0.001 0.001"/>
+        <mesh filename="file://$(find cookobot_gazebo)/robot_description/urdf/meshes/sensors/lds.stl" scale="0.001 0.001 0.001"/>
       </geometry>
       <material name="dark"/>
@@ -191,4 +191,4 @@
   </joint>
 <!-- ARM -->
-    <xacro:include filename="$(find cookobot-arm)/robot_description/urdf/turtlebot_arm.xacro"/>
+    <xacro:include filename="$(find cookobot_gazebo)/robot_description/urdf/turtlebot_arm.xacro"/>
 </robot>

File: cookobot_gazebo/robot_description/urdf/turtlebot_arm.xacro (robot description, xacro)
@@ -35,5 +35,5 @@
             <origin rpy="0 0 0" xyz=" 0 0 0 " />
             <geometry>
-                <mesh filename="file://$(find cookobot-arm)/robot_description/urdf/meshes/arm/ax12_box.stl" scale="0.001 0.001 0.001" />
+                <mesh filename="file://$(find cookobot_gazebo)/robot_description/urdf/meshes/arm/ax12_box.stl" scale="0.001 0.001 0.001" />
             </geometry>
             <material name="Black" />
@@ -63,5 +63,5 @@
             <origin rpy="0 0 0" xyz=" 0 0 0 " />
             <geometry>
-                <mesh filename="file://$(find cookobot-arm)/robot_description/urdf/meshes/arm/F3.stl" scale="0.001 0.001 0.001" />
+                <mesh filename="file://$(find cookobot_gazebo)/robot_description/urdf/meshes/arm/F3.stl" scale="0.001 0.001 0.001" />
             </geometry>
             <material name="White" />
@@ -89,5 +89,5 @@
             <origin rpy="0 0 0" xyz=" 0 0 0 " />
             <geometry>
-                <mesh filename="file://$(find cookobot-arm)/robot_description/urdf/meshes/arm/ax12_box.stl" scale="0.001 0.001 0.001" />
+                <mesh filename="file://$(find cookobot_gazebo)/robot_description/urdf/meshes/arm/ax12_box.stl" scale="0.001 0.001 0.001" />
             </geometry>
             <material name="Black" />
@@ -117,5 +117,5 @@
             <origin rpy="0 0 0" xyz=" 0 0 0 " />
             <geometry>
-                <mesh filename="file://$(find cookobot-arm)/robot_description/urdf/meshes/arm/F4.stl" scale="0.001 0.001 0.001" />
+                <mesh filename="file://$(find cookobot_gazebo)/robot_description/urdf/meshes/arm/F4.stl" scale="0.001 0.001 0.001" />
             </geometry>
             <material name="White" />
@@ -143,5 +143,5 @@
             <origin rpy="0 0 0" xyz=" 0 0 0 " />
             <geometry>
-                <mesh filename="file://$(find cookobot-arm)/robot_description/urdf/meshes/arm/F10.stl" scale="0.001 0.001 0.001" />
+                <mesh filename="file://$(find cookobot_gazebo)/robot_description/urdf/meshes/arm/F10.stl" scale="0.001 0.001 0.001" />
             </geometry>
             <material name="White" />
@@ -169,5 +169,5 @@
             <origin rpy="0 0 0" xyz=" 0 0 0 " />
             <geometry>
-                <mesh filename="file://$(find cookobot-arm)/robot_description/urdf/meshes/arm/F10.stl" scale="0.001 0.001 0.001" />
+                <mesh filename="file://$(find cookobot_gazebo)/robot_description/urdf/meshes/arm/F10.stl" scale="0.001 0.001 0.001" />
             </geometry>
             <material name="White" />
@@ -195,5 +195,5 @@
             <origin rpy="0 0 0" xyz=" 0 0 0 " />
             <geometry>
-                <mesh filename="file://$(find cookobot-arm)/robot_description/urdf/meshes/arm/F10.stl" scale="0.001 0.001 0.001" />
+                <mesh filename="file://$(find cookobot_gazebo)/robot_description/urdf/meshes/arm/F10.stl" scale="0.001 0.001 0.001" />
             </geometry>
             <material name="White" />
@@ -221,5 +221,5 @@
             <origin rpy="0 0 0" xyz=" 0 0 0 " />
             <geometry>
-                <mesh filename="file://$(find cookobot-arm)/robot_description/urdf/meshes/arm/F3.stl" scale="0.001 0.001 0.001" />
+                <mesh filename="file://$(find cookobot_gazebo)/robot_description/urdf/meshes/arm/F3.stl" scale="0.001 0.001 0.001" />
             </geometry>
             <material name="White" />
@@ -247,5 +247,5 @@
             <origin rpy="0 0 0" xyz=" 0 0 0 " />
             <geometry>
-                <mesh filename="file://$(find cookobot-arm)/robot_description/urdf/meshes/arm/ax12_box.stl" scale="0.001 0.001 0.001" />
+                <mesh filename="file://$(find cookobot_gazebo)/robot_description/urdf/meshes/arm/ax12_box.stl" scale="0.001 0.001 0.001" />
             </geometry>
             <material name="Black" />
@@ -275,5 +275,5 @@
             <origin rpy="0 0 0" xyz=" 0 0 0 " />
             <geometry>
-                <mesh filename="file://$(find cookobot-arm)/robot_description/urdf/meshes/arm/F4.stl" scale="0.001 0.001 0.001" />
+                <mesh filename="file://$(find cookobot_gazebo)/robot_description/urdf/meshes/arm/F4.stl" scale="0.001 0.001 0.001" />
             </geometry>
             <material name="White" />
@@ -301,5 +301,5 @@
             <origin rpy="0 0 0" xyz=" 0 0 0 " />
             <geometry>
-                <mesh filename="file://$(find cookobot-arm)/robot_description/urdf/meshes/arm/F10.stl" scale="0.001 0.001 0.001" />
+                <mesh filename="file://$(find cookobot_gazebo)/robot_description/urdf/meshes/arm/F10.stl" scale="0.001 0.001 0.001" />
             </geometry>
             <material name="White" />
@@ -327,5 +327,5 @@
             <origin rpy="0 0 0" xyz=" 0 0 0 " />
             <geometry>
-                <mesh filename="file://$(find cookobot-arm)/robot_description/urdf/meshes/arm/F10.stl" scale="0.001 0.001 0.001" />
+                <mesh filename="file://$(find cookobot_gazebo)/robot_description/urdf/meshes/arm/F10.stl" scale="0.001 0.001 0.001" />
             </geometry>
             <material name="White" />
@@ -353,5 +353,5 @@
             <origin rpy="0 0 0" xyz=" 0 0 0 " />
             <geometry>
-                <mesh filename="file://$(find cookobot-arm)/robot_description/urdf/meshes/arm/F10.stl" scale="0.001 0.001 0.001" />
+                <mesh filename="file://$(find cookobot_gazebo)/robot_description/urdf/meshes/arm/F10.stl" scale="0.001 0.001 0.001" />
             </geometry>
             <material name="White" />
@@ -379,5 +379,5 @@
             <origin rpy="0 0 0" xyz=" 0 0 0 " />
             <geometry>
-                <mesh filename="file://$(find cookobot-arm)/robot_description/urdf/meshes/arm/F3.stl" scale="0.001 0.001 0.001" />
+                <mesh filename="file://$(find cookobot_gazebo)/robot_description/urdf/meshes/arm/F3.stl" scale="0.001 0.001 0.001" />
             </geometry>
             <material name="White" />
@@ -405,5 +405,5 @@
             <origin rpy="0 0 0" xyz=" 0 0 0 " />
             <geometry>
-                <mesh filename="file://$(find cookobot-arm)/robot_description/urdf/meshes/arm/ax12_box.stl" scale="0.001 0.001 0.001" />
+                <mesh filename="file://$(find cookobot_gazebo)/robot_description/urdf/meshes/arm/ax12_box.stl" scale="0.001 0.001 0.001" />
             </geometry>
             <material name="Black" />
@@ -433,5 +433,5 @@
             <origin rpy="0 0 0" xyz=" 0 0 0 " />
             <geometry>
-                <mesh filename="file://$(find cookobot-arm)/robot_description/urdf/meshes/arm/F2.stl" scale="0.001 0.001 0.001" />
+                <mesh filename="file://$(find cookobot_gazebo)/robot_description/urdf/meshes/arm/F2.stl" scale="0.001 0.001 0.001" />
             </geometry>
             <material name="White" />
@@ -459,5 +459,5 @@
             <origin rpy="0 0 0" xyz=" 0 0 0 " />
             <geometry>
-                <mesh filename="file://$(find cookobot-arm)/robot_description/urdf/meshes/arm/F3.stl" scale="0.001 0.001 0.001" />
+                <mesh filename="file://$(find cookobot_gazebo)/robot_description/urdf/meshes/arm/F3.stl" scale="0.001 0.001 0.001" />
             </geometry>
             <material name="White" />
@@ -485,5 +485,5 @@
             <origin rpy="0 0 0" xyz=" 0 0 0 " />
             <geometry>
-                <mesh filename="file://$(find cookobot-arm)/robot_description/urdf/meshes/arm/ax12_box.stl" scale="0.001 0.001 0.001" />
+                <mesh filename="file://$(find cookobot_gazebo)/robot_description/urdf/meshes/arm/ax12_box.stl" scale="0.001 0.001 0.001" />
             </geometry>
             <material name="Black" />
@@ -513,5 +513,5 @@
             <origin rpy="0 0 0" xyz=" 0 0 0 " />
             <geometry>
-                <mesh filename="file://$(find cookobot-arm)/robot_description/urdf/meshes/arm/F2.stl" scale="0.001 0.001 0.001" />
+                <mesh filename="file://$(find cookobot_gazebo)/robot_description/urdf/meshes/arm/F2.stl" scale="0.001 0.001 0.001" />
             </geometry>
             <material name="White" />
@@ -539,5 +539,5 @@
             <origin rpy="0 0 0" xyz=" 0 0 0 " />
             <geometry>
-                <mesh filename="file://$(find cookobot-arm)/robot_description/urdf/meshes/arm/turtlebot_finger.stl" scale="0.001 0.001 0.001" />
+                <mesh filename="file://$(find cookobot_gazebo)/robot_description/urdf/meshes/arm/turtlebot_finger.stl" scale="0.001 0.001 0.001" />
             </geometry>
             <material name="Green" />
@@ -565,5 +565,5 @@
             <origin rpy="0 0 0" xyz=" 0 0 0 " />
             <geometry>
-                <mesh filename="file://$(find cookobot-arm)/robot_description/urdf/meshes/arm/F3.stl" scale="0.001 0.001 0.001" />
+                <mesh filename="file://$(find cookobot_gazebo)/robot_description/urdf/meshes/arm/F3.stl" scale="0.001 0.001 0.001" />
             </geometry>
             <material name="White" />
@@ -591,5 +591,5 @@
             <origin rpy="0 0 0" xyz=" 0 0 0 " />
             <geometry>
-                <mesh filename="file://$(find cookobot-arm)/robot_description/urdf/meshes/arm/turtlebot_finger.stl" scale="0.001 0.001 0.001" />
+                <mesh filename="file://$(find cookobot_gazebo)/robot_description/urdf/meshes/arm/turtlebot_finger.stl" scale="0.001 0.001 0.001" />
             </geometry>
             <material name="Green" />

File: cookobot_gazebo/robot_description/urdf/turtlebot_gripper.xacro (robot description, xacro)
@@ -28,5 +28,5 @@
         <origin xyz=" 0 0 0 " rpy="0 0 0"/>
         <geometry>
-          <mesh filename="file://$(find cookobot-arm)/robot_description/urdf/meshes/F2.stl" scale="${M_SCALE} ${M_SCALE} ${M_SCALE}"/>
+          <mesh filename="file://$(find cookobot_gazebo)/robot_description/urdf/meshes/F2.stl" scale="${M_SCALE} ${M_SCALE} ${M_SCALE}"/>
         </geometry>
         <material name="${color}"/>
