Commit message: Add tray and remove finger

File: cookobot_gazebo/robot_description/urdf/turtlebot_arm.xacro (robot description, xacro)
@@ -2,17 +2,17 @@
 <!-- Arm description for Turtlebot Arm and PhantomX Pincher arm -->
 <robot xmlns:xacro="http://ros.org/wiki/xacro">
-  <material name="White">
-    <color rgba="0.87 0.90 0.87 1.0"/>
-  </material>
-  <material name="Black">
-    <color rgba="0.08 0.08 0.08 1.0"/>
-  </material>
-  <material name="Gray">
-    <color rgba="0.2 0.2 0.21 1.0"/>
-  </material>
-  <material name="Green">
-    <color rgba="0.22 0.32 0.14 1.0"/>
-  </material>
- <link name="arm_base_link" />
+    <material name="White">
+        <color rgba="0.87 0.90 0.87 1.0"/>
+    </material>
+    <material name="Black">
+        <color rgba="0.08 0.08 0.08 1.0"/>
+    </material>
+    <material name="Gray">
+        <color rgba="0.2 0.2 0.21 1.0"/>
+    </material>
+    <material name="Green">
+        <color rgba="0.22 0.32 0.14 1.0"/>
+    </material>
+    <link name="arm_base_link" />
     <joint name="arm_base_joint" type="fixed">
         <origin xyz="${origin_arm}" />
@@ -26,9 +26,9 @@
     </joint>
     <link name="arm_shoulder_pan_servo_link">
-	<inertial>
+        <inertial>
             <mass value="0.055" />
             <origin xyz="0 0 0" />
             <inertia ixx="0.000017012" ixy="0.0" ixz="0.0" iyy="0.000013258" iyz="0.0" izz="0.000009483" />
-	    <dynamics damping="0.5" friction="0.1"/>
+            <dynamics damping="0.5" friction="0.1"/>
         </inertial>
         <visual>
@@ -58,5 +58,5 @@
             <origin xyz="0 0 0" />
             <inertia ixx="4.70666666667e-07" ixy="0" ixz="0" iyy="1.37933333333e-06" iyz="0" izz="1.01666666667e-06" />
-	    <dynamics damping="0.5" friction="0.1"/>
+            <dynamics damping="0.5" friction="0.1"/>
         </inertial>
         <visual>
@@ -80,10 +80,10 @@
     </joint>
     <link name="arm_shoulder_lift_servo_link">
-    <inertial>
+        <inertial>
             <mass value="0.055" />
             <origin xyz="0 0 0" />
             <inertia ixx="0.000017012" ixy="0.0" ixz="0.0" iyy="0.000013258" iyz="0.0" izz="0.000009483" />
-	    <dynamics damping="0.5" friction="0.1"/>
-    </inertial>
+            <dynamics damping="0.5" friction="0.1"/>
+        </inertial>
         <visual>
             <origin rpy="0 0 0" xyz=" 0 0 0 " />
@@ -108,9 +108,9 @@
     </joint>
     <link name="arm_shoulder_lift_link">
-    <inertial>
+        <inertial>
             <mass value="0.016" />
             <origin xyz="0 0 0" />
             <inertia ixx="6.67866666667e-06" ixy="0" ixz="0" iyy="4.18166666667e-06" iyz="0" izz="8.76966666667e-06" />
-	    <dynamics damping="0.5" friction="0.1"/>
+            <dynamics damping="0.5" friction="0.1"/>
         </inertial>
         <visual>
@@ -134,9 +134,9 @@
     </joint>
     <link name="arm_shoulder_F10_0_link">
-    <inertial>
+        <inertial>
             <mass value="0.004" />
             <origin xyz="0 0 0" />
             <inertia ixx="2.13666666667e-07" ixy="0" ixz="0" iyy="6.89666666667e-07" iyz="0" izz="4.86666666667e-07" />
-	    <dynamics damping="0.5" friction="0.1"/>
+            <dynamics damping="0.5" friction="0.1"/>
         </inertial>
         <visual>
@@ -160,9 +160,9 @@
     </joint>
     <link name="arm_shoulder_F10_1_link">
-    <inertial>
+        <inertial>
             <mass value="0.004" />
             <origin xyz="0 0 0" />
             <inertia ixx="2.13666666667e-07" ixy="0" ixz="0" iyy="6.89666666667e-07" iyz="0" izz="4.86666666667e-07" />
-	    <dynamics damping="0.5" friction="0.1"/>
+            <dynamics damping="0.5" friction="0.1"/>
         </inertial>
         <visual>
@@ -186,9 +186,9 @@
     </joint>
     <link name="arm_shoulder_F10_2_link">
-    <inertial>
+        <inertial>
             <mass value="0.004" />
             <origin xyz="0 0 0" />
             <inertia ixx="2.13666666667e-07" ixy="0" ixz="0" iyy="6.89666666667e-07" iyz="0" izz="4.86666666667e-07" />
-	    <dynamics damping="0.5" friction="0.1"/>
+            <dynamics damping="0.5" friction="0.1"/>
         </inertial>
         <visual>
@@ -212,9 +212,9 @@
     </joint>
     <link name="arm_shoulder_F3_0_link">
-   <inertial>
+        <inertial>
             <mass value="0.005" />
             <origin xyz="0 0 0" />
             <inertia ixx="2.94166666667e-07" ixy="0" ixz="0" iyy="8.62083333333e-07" iyz="0" izz="6.35416666667e-07" />
-	    <dynamics damping="0.5" friction="0.1"/>
+            <dynamics damping="0.5" friction="0.1"/>
         </inertial>
         <visual>
@@ -238,9 +238,9 @@
     </joint>
     <link name="arm_elbow_flex_servo_link">
-   <inertial>
+        <inertial>
             <mass value="0.055" />
             <origin xyz="0 0 0" />
             <inertia ixx="0.000017012" ixy="0.0" ixz="0.0" iyy="0.000013258" iyz="0.0" izz="0.000009483" />
-	    <dynamics damping="0.5" friction="0.1"/>
+            <dynamics damping="0.5" friction="0.1"/>
         </inertial>
         <visual>
@@ -266,9 +266,9 @@
     </joint>
     <link name="arm_elbow_flex_link">
-   <inertial>
+        <inertial>
             <mass value="0.016" />
             <origin xyz="0 0 0" />
             <inertia ixx="6.67866666667e-06" ixy="0" ixz="0" iyy="4.18166666667e-06" iyz="0" izz="8.76966666667e-06" />
-	    <dynamics damping="0.5" friction="0.1"/>
+            <dynamics damping="0.5" friction="0.1"/>
         </inertial>
         <visual>
@@ -292,9 +292,9 @@
     </joint>
     <link name="arm_elbow_F10_0_link">
-    <inertial>
+        <inertial>
             <mass value="0.004" />
             <origin xyz="0 0 0" />
             <inertia ixx="2.13666666667e-07" ixy="0" ixz="0" iyy="6.89666666667e-07" iyz="0" izz="4.86666666667e-07" />
-	    <dynamics damping="0.5" friction="0.1"/>
+            <dynamics damping="0.5" friction="0.1"/>
         </inertial>
         <visual>
@@ -318,9 +318,9 @@
     </joint>
     <link name="arm_elbow_F10_1_link">
-    <inertial>
+        <inertial>
             <mass value="0.004" />
             <origin xyz="0 0 0" />
             <inertia ixx="2.13666666667e-07" ixy="0" ixz="0" iyy="6.89666666667e-07" iyz="0" izz="4.86666666667e-07" />
-	    <dynamics damping="0.5" friction="0.1"/>
+            <dynamics damping="0.5" friction="0.1"/>
         </inertial>
         <visual>
@@ -344,9 +344,9 @@
     </joint>
     <link name="arm_elbow_F10_2_link">
-    <inertial>
+        <inertial>
             <mass value="0.004" />
             <origin xyz="0 0 0" />
             <inertia ixx="2.13666666667e-07" ixy="0" ixz="0" iyy="6.89666666667e-07" iyz="0" izz="4.86666666667e-07" />
-	    <dynamics damping="0.5" friction="0.1"/>
+            <dynamics damping="0.5" friction="0.1"/>
         </inertial>
         <visual>
@@ -370,9 +370,9 @@
     </joint>
     <link name="arm_elbow_F3_0_link">
-    <inertial>
+        <inertial>
             <mass value="0.005" />
             <origin xyz="0 0 0" />
             <inertia ixx="2.94166666667e-07" ixy="0" ixz="0" iyy="8.62083333333e-07" iyz="0" izz="6.35416666667e-07" />
-	    <dynamics damping="0.5" friction="0.1"/>
+            <dynamics damping="0.5" friction="0.1"/>
         </inertial>
         <visual>
@@ -396,9 +396,9 @@
     </joint>
     <link name="arm_wrist_flex_servo_link">
-   <inertial>
+        <inertial>
             <mass value="0.055" />
             <origin xyz="0 0 0" />
             <inertia ixx="0.000017012" ixy="0.0" ixz="0.0" iyy="0.000013258" iyz="0.0" izz="0.000009483" />
-	    <dynamics damping="0.5" friction="0.1"/>
+            <dynamics damping="0.5" friction="0.1"/>
         </inertial>
         <visual>
@@ -424,9 +424,9 @@
     </joint>
     <link name="arm_wrist_flex_link">
-<inertial>
+        <inertial>
             <mass value="0.01" />
             <origin xyz="0 0 0" />
             <inertia ixx="1.69270833333e-06" ixy="0" ixz="0" iyy="2.48104166667e-06" iyz="0" izz="3.13208333333e-06" />
-	    <dynamics damping="0.5" friction="0.1"/>
+            <dynamics damping="0.5" friction="0.1"/>
         </inertial>
         <visual>
@@ -450,9 +450,9 @@
     </joint>
     <link name="arm_wrist_F3_0_link">
-    <inertial>
+        <inertial>
             <mass value="0.005" />
             <origin xyz="0 0 0" />
             <inertia ixx="2.94166666667e-07" ixy="0" ixz="0" iyy="8.62083333333e-07" iyz="0" izz="6.35416666667e-07" />
-	    <dynamics damping="0.5" friction="0.1"/>
+            <dynamics damping="0.5" friction="0.1"/>
         </inertial>
         <visual>
@@ -476,9 +476,9 @@
     </joint>
     <link name="gripper_servo_link">
-   <inertial>
+        <inertial>
             <mass value="0.055" />
             <origin xyz="0 0 0" />
             <inertia ixx="0.000017012" ixy="0.0" ixz="0.0" iyy="0.000013258" iyz="0.0" izz="0.000009483" />
-	    <dynamics damping="0.5" friction="0.1"/>
+            <dynamics damping="0.5" friction="0.1"/>
         </inertial>
         <visual>
@@ -505,5 +505,5 @@
     </joint>
     <link name="gripper_active_link">
-    <inertial>
+        <inertial>
             <mass value="0.010" />
             <origin xyz="0 0 0" />
@@ -530,66 +530,14 @@
     </joint>
     <link name="gripper_active_finger_link">
-<inertial>
+        <inertial>
             <mass value="0.015" />
             <origin xyz="0 0 0" />
             <inertia ixx="8.129225e-06" ixy="0" ixz="0" iyy="9.469562625e-06" iyz="0" izz="2.271562625e-06" />
-	    <dynamics damping="0.5" friction="0.1"/>
-        </inertial>
-        <visual>
-            <origin rpy="0 0 0" xyz=" 0 0 0 " />
-            <geometry>
-                <mesh filename="file://$(find cookobot_gazebo)/robot_description/urdf/meshes/arm/turtlebot_finger.stl" scale="0.001 0.001 0.001" />
-            </geometry>
-            <material name="Green" />
-        </visual>
-        <collision>
-            <origin rpy="0 0 0" xyz="0.02645 0.0 -0.00655" />
-            <geometry>
-                <box size="0.0783 0.03801 0.0193" />
-            </geometry>
-        </collision>
-    </link>
-    <joint name="gripper_static_joint" type="fixed">
-        <origin rpy="0 3.14159 0" xyz="0 0 -0.0415" />
-        <parent link="gripper_servo_link" />
-        <child link="gripper_static_link" />
-    </joint>
-    <link name="gripper_static_link">
-<inertial>
-            <mass value="0.005" />
-            <origin xyz="0 0 0" />
-            <inertia ixx="2.94166666667e-07" ixy="0" ixz="0" iyy="8.62083333333e-07" iyz="0" izz="6.35416666667e-07" />
-	    <dynamics damping="0.5" friction="0.1"/>
-        </inertial>
-        <visual>
-            <origin rpy="0 0 0" xyz=" 0 0 0 " />
-            <geometry>
-                <mesh filename="file://$(find cookobot_gazebo)/robot_description/urdf/meshes/arm/F3.stl" scale="0.001 0.001 0.001" />
-            </geometry>
-            <material name="White" />
-        </visual>
-        <collision>
-            <origin rpy="0 0 0" xyz="0.0 0.0 -0.0045" />
-            <geometry>
-                <box size="0.025 0.038 0.009" />
-            </geometry>
-        </collision>
-    </link>
-    <joint name="gripper_static_finger_joint" type="fixed">
-        <origin rpy="0 0 3.14159" xyz="0 0 0" />
-        <parent link="gripper_static_link" />
-        <child link="gripper_static_finger_link" />
-    </joint>
-    <link name="gripper_static_finger_link">
-<inertial>
-            <mass value="0.015" />
-            <origin xyz="0 0 0" />
-            <inertia ixx="8.129225e-06" ixy="0" ixz="0" iyy="9.469562625e-06" iyz="0" izz="2.271562625e-06" />
-	    <dynamics damping="0.5" friction="0.1"/>
-        </inertial>
-        <visual>
-            <origin rpy="0 0 0" xyz=" 0 0 0 " />
-            <geometry>
-                <mesh filename="file://$(find cookobot_gazebo)/robot_description/urdf/meshes/arm/turtlebot_finger.stl" scale="0.001 0.001 0.001" />
+            <dynamics damping="0.5" friction="0.1"/>
+        </inertial>
+        <visual>
+            <origin rpy="0 0 0" xyz=" 0 0 0 " />
+            <geometry>
+                <mesh filename="file://$(find cookobot_gazebo)/robot_description/urdf/meshes/tray_bottles.stl" scale="0.001 0.001 0.001" />
             </geometry>
             <material name="Green" />
@@ -604,57 +552,53 @@
     <!-- shoulder pan joint-->
     <dynamixel_AX12_fixed parent="arm_base_link" name="arm_shoulder_pan_servo">
-      <origin xyz="0 0 0" rpy="${M_PI/2} 0 ${M_PI/2}"/>
+        <origin xyz="0 0 0" rpy="${M_PI/2} 0 ${M_PI/2}"/>
     </dynamixel_AX12_fixed>
-    <bioloid_F3_revolute parent="arm_shoulder_pan_servo_link" name="arm_shoulder_pan" color="${color}"
-                         vlimit="${joints_vlimit}" llimit="${pan_llimit}" ulimit="${pan_ulimit}">
-      <origin xyz="0 ${AX12_WIDTH/2} 0" rpy="${-M_PI/2} ${M_PI/2} ${M_PI}"/>
+    <bioloid_F3_revolute parent="arm_shoulder_pan_servo_link" name="arm_shoulder_pan" color="${color}" vlimit="${joints_vlimit}" llimit="${pan_llimit}" ulimit="${pan_ulimit}">
+        <origin xyz="0 ${AX12_WIDTH/2} 0" rpy="${-M_PI/2} ${M_PI/2} ${M_PI}"/>
     </bioloid_F3_revolute> -->
     <!-- shoulder lift joint -->
     <dynamixel_AX12_fixed parent="arm_shoulder_pan_link" name="arm_shoulder_lift_servo">
-      <origin xyz="0 0 ${-AX12_HEIGHT-F10_HEIGHT+0.001}" rpy="0 ${M_PI} 0"/>
+        <origin xyz="0 0 ${-AX12_HEIGHT-F10_HEIGHT+0.001}" rpy="0 ${M_PI} 0"/>
     </dynamixel_AX12_fixed>
-    <bioloid_F4_revolute parent="arm_shoulder_lift_servo_link" name="arm_shoulder_lift" color="${color}"
-                         vlimit="${joints_vlimit}" llimit="${shoulder_llimit}" ulimit="${shoulder_ulimit}">
-      <origin xyz="0 0 0" rpy="0 0 0"/>
+    <bioloid_F4_revolute parent="arm_shoulder_lift_servo_link" name="arm_shoulder_lift" color="${color}" vlimit="${joints_vlimit}" llimit="${shoulder_llimit}" ulimit="${shoulder_ulimit}">
+        <origin xyz="0 0 0" rpy="0 0 0"/>
     </bioloid_F4_revolute>
     <bioloid_F10_fixed parent="arm_shoulder_lift_link" name="arm_shoulder_F10_0" color="${color}">
-      <origin xyz="0 0 ${F4_HEIGHT+F10_HEIGHT/2}" rpy="0 0 0"/>
+        <origin xyz="0 0 ${F4_HEIGHT+F10_HEIGHT/2}" rpy="0 0 0"/>
     </bioloid_F10_fixed>
     <bioloid_F10_fixed parent="arm_shoulder_F10_0_link" name="arm_shoulder_F10_1" color="${color}">
-      <origin xyz="0 0 ${F10_HEIGHT}" rpy="0 0 0"/>
+        <origin xyz="0 0 ${F10_HEIGHT}" rpy="0 0 0"/>
     </bioloid_F10_fixed>
     <bioloid_F10_fixed parent="arm_shoulder_F10_1_link" name="arm_shoulder_F10_2" color="${color}">
-      <origin xyz="0 0 ${F10_HEIGHT}" rpy="0 0 0"/>
+        <origin xyz="0 0 ${F10_HEIGHT}" rpy="0 0 0"/>
     </bioloid_F10_fixed>
     <bioloid_F3_fixed parent="arm_shoulder_F10_2_link" name="arm_shoulder_F3_0" color="${color}">
-      <origin xyz="0 0 ${F10_HEIGHT/2}" rpy="0 ${M_PI} 0"/>
+        <origin xyz="0 0 ${F10_HEIGHT/2}" rpy="0 ${M_PI} 0"/>
     </bioloid_F3_fixed> -->
     <!-- elbow joint -->
     <dynamixel_AX12_fixed parent="arm_shoulder_F3_0_link" name="arm_elbow_flex_servo">
-      <origin xyz="0 0 ${-AX12_HEIGHT-F10_HEIGHT+0.001}" rpy="0 ${M_PI} 0"/>
+        <origin xyz="0 0 ${-AX12_HEIGHT-F10_HEIGHT+0.001}" rpy="0 ${M_PI} 0"/>
     </dynamixel_AX12_fixed>
-    <bioloid_F4_revolute parent="arm_elbow_flex_servo_link" name="arm_elbow_flex" color="${color}"
-                         vlimit="${joints_vlimit}" llimit="${elbow_llimit}" ulimit="${elbow_ulimit}">
-      <origin xyz="0 0 0" rpy="0 0 0"/>
+    <bioloid_F4_revolute parent="arm_elbow_flex_servo_link" name="arm_elbow_flex" color="${color}" vlimit="${joints_vlimit}" llimit="${elbow_llimit}" ulimit="${elbow_ulimit}">
+        <origin xyz="0 0 0" rpy="0 0 0"/>
     </bioloid_F4_revolute>
     <bioloid_F10_fixed parent="arm_elbow_flex_link" name="arm_elbow_F10_0" color="${color}">
-      <origin xyz="0 0 ${F4_HEIGHT+F10_HEIGHT/2}" rpy="0 0 0"/>
+        <origin xyz="0 0 ${F4_HEIGHT+F10_HEIGHT/2}" rpy="0 0 0"/>
     </bioloid_F10_fixed>
     <bioloid_F10_fixed parent="arm_elbow_F10_0_link" name="arm_elbow_F10_1" color="${color}">
-      <origin xyz="0 0 ${F10_HEIGHT}" rpy="0 0 0"/>
+        <origin xyz="0 0 ${F10_HEIGHT}" rpy="0 0 0"/>
     </bioloid_F10_fixed>
     <bioloid_F10_fixed parent="arm_elbow_F10_1_link" name="arm_elbow_F10_2" color="${color}">
-      <origin xyz="0 0 ${F10_HEIGHT}" rpy="0 0 0"/>
+        <origin xyz="0 0 ${F10_HEIGHT}" rpy="0 0 0"/>
     </bioloid_F10_fixed>
     <bioloid_F3_fixed parent="arm_elbow_F10_2_link" name="arm_elbow_F3_0" color="${color}">
-      <origin xyz="0 0 ${F10_HEIGHT/2}" rpy="0 ${M_PI} 0"/>
+        <origin xyz="0 0 ${F10_HEIGHT/2}" rpy="0 ${M_PI} 0"/>
     </bioloid_F3_fixed>
-  <!-- wrist joint -->
+    <!-- wrist joint -->
     <dynamixel_AX12_fixed parent="arm_elbow_F3_0_link" name="arm_wrist_flex_servo">
-      <origin xyz="0 0 ${-AX12_HEIGHT-F10_HEIGHT+0.001}" rpy="0 ${M_PI} 0"/>
+        <origin xyz="0 0 ${-AX12_HEIGHT-F10_HEIGHT+0.001}" rpy="0 ${M_PI} 0"/>
     </dynamixel_AX12_fixed>
-    <bioloid_F2_revolute parent="arm_wrist_flex_servo_link" name="arm_wrist_flex" color="${color}"
-                         vlimit="${joints_vlimit}" llimit="${wrist_llimit}" ulimit="${wrist_ulimit}">
-      <origin xyz="0 0 0" rpy="0 0 0"/>
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