Commit message: Change tray color

File: cookobot_gazebo/robot_description/urdf/turtlebot3_burger_arm.gazebo.xacro (robot description, xacro)
@@ -167,5 +167,5 @@
     </gazebo>
       <gazebo reference="gripper_active_finger_link">
-        <material>Gazebo/Green</material>
+        <material>Gazebo/Grey1</material>
         <selfCollide>true</selfCollide>
         <turnGravityOff>true</turnGravityOff>
